File: Daughterboardv2.kicad_pcb (KiCad board)
At the start: 2 copper layers, 49.5 x 25 mm, 15 parts, among them J1 Conn_01x06_Male, J2 Conn_01x01, J3 Conn_01x05_Pin, J4 Conn_01x05_Pin, U1 XIAO-ESP32C3, U2 TJA1042T-3

Commit message: add second option for CAN transorb
Parts:
- added D2: PESD1CAN, Package_TO_SOT_SMD:SOT-23, B.Cu at (140.6, 97.6)
Routing:
- net /CANH: track 40.8 -> 45.8 mm, vias 0 -> 2
- net /CANL: track 43.0 -> 45.3 mm
Changed lines of the file:
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@@
+    )
+  )
+  (footprint "Package_TO_SOT_SMD:SOT-23" (layer "B.Cu")
+    (at 140.6 97.6 90)
+    (descr "SOT, 3 Pin (https://www.jedec.org/system/files/docs/to-236h.pdf variant AB), generated with kicad-footprint-generator ipc_gullwing_generator.py")
+    (tags "SOT TO_SOT_SMD")
+    (property "Sheetfile" "Daughterboardv2.kicad_sch")
+    (property "Sheetname" "")
+    (property "ki_description" "Bidirectional dual transient-voltage-suppression diode, center on pin 3")
+    (property "ki_keywords" "diode TVS thyrector")
+    (attr smd)
+    (fp_text reference "D2" (at 0 2.4 90) (layer "B.SilkS")
+        (effects (font (size 1 1) (thickness 0.15)) (justify mirror))
+    )
+    (fp_text value "PESD1CAN" (at 0 -2.4 90) (layer "B.Fab")
+        (effects (font (size 1 1) (thickness 0.15)) (justify mirror))
+    )
+    (fp_text user "${REFERENCE}" (at 0 0 90) (layer "B.Fab")
+        (effects (font (size 0.32 0.32) (thickness 0.05)) (justify mirror))
+    )
+    (fp_line (start 0 -1.56) (end -0.65 -1.56)
+      (stroke (width 0.12) (type solid)) (layer "B.SilkS"))
+    (fp_line (start 0 -1.56) (end 0.65 -1.56)
+      (stroke (width 0.12) (type solid)) (layer "B.SilkS"))
+    (fp_line (start 0 1.56) (end -1.675 1.56)
+      (stroke (width 0.12) (type solid)) (layer "B.SilkS"))
+    (fp_line (start 0 1.56) (end 0.65 1.56)
+      (stroke (width 0.12) (type solid)) (layer "B.SilkS"))
+    (fp_line (start -1.92 -1.7) (end 1.92 -1.7)
+      (stroke (width 0.05) (type solid)) (layer "B.CrtYd"))
+    (fp_line (start -1.92 1.7) (end -1.92 -1.7)
+      (stroke (width 0.05) (type solid)) (layer "B.CrtYd"))
+    (fp_line (start 1.92 -1.7) (end 1.92 1.7)
+      (stroke (width 0.05) (type solid)) (layer "B.CrtYd"))
+    (fp_line (start 1.92 1.7) (end -1.92 1.7)
+      (stroke (width 0.05) (type solid)) (layer "B.CrtYd"))
+    (fp_line (start -0.65 -1.45) (end -0.65 1.125)
+      (stroke (width 0.1) (type solid)) (layer "B.Fab"))
+    (fp_line (start -0.65 1.125) (end -0.325 1.45)
+      (stroke (width 0.1) (type solid)) (layer "B.Fab"))
+    (fp_line (start -0.325 1.45) (end 0.65 1.45)
+      (stroke (width 0.1) (type solid)) (layer "B.Fab"))
+    (fp_line (start 0.65 -1.45) (end -0.65 -1.45)
+      (stroke (width 0.1) (type solid)) (layer "B.Fab"))
+    (fp_line (start 0.65 1.45) (end 0.65 -1.45)
+      (stroke (width 0.1) (type solid)) (layer "B.Fab"))
+    (pad "1" smd roundrect (at -0.9375 0.95 90) (size 1.475 0.6) (layers "B.Cu" "B.Paste" "B.Mask") (roundrect_rratio 0.25)
+      (net 3 "/CANH") (pinfunction "A1") (pintype "passive"))
+    (pad "2" smd roundrect (at -0.9375 -0.95 90) (size 1.475 0.6) (layers "B.Cu" "B.Paste" "B.Mask") (roundrect_rratio 0.25)
+      (net 4 "/CANL") (pinfunction "A2") (pintype "passive"))
+    (pad "3" smd roundrect (at 0.9375 0 90) (size 1.475 0.6) (layers "B.Cu" "B.Paste" "B.Mask") (roundrect_rratio 0.25)
+      (net 2 "GND") (pinfunction "common") (pintype "passive"))
+    (model "${KICAD6_3DMODEL_DIR}/Package_TO_SOT_SMD.3dshapes/SOT-23.wrl"
+      (offset (xyz 0 0 0))
+      (scale (xyz 1 1 1))
+      (rotate (xyz 0 0 0))
     )
   )
@@
   (via (at 131 109.8) (size 0.8) (drill 0.4) (layers "F.Cu" "B.Cu") (free) (net 2))
   (via (at 172 110.5) (size 0.8) (drill 0.4) (layers "F.Cu" "B.Cu") (free) (net 2))
+  (segment (start 143.8 99.2) (end 143.8 101.7) (width 0.5) (layer "F.Cu") (net 3))
+  (via (at 143.8 99.2) (size 0.8) (drill 0.4) (layers "F.Cu" "B.Cu") (net 3))
+  (via (at 143.589143 101.675926) (size 0.8) (drill 0.4) (layers "F.Cu" "B.Cu") (net 3))
   (segment (start 174.5 102.25) (end 174.25 102) (width 0.2) (layer "B.Cu") (net 3))
   (segment (start 151.9 98.5) (end 151.9 100.8) (width 0.5) (layer "B.Cu") (net 3))
-  (segment (start 141.3 101.7) (end 151 101.7) (width 0.5) (layer "B.Cu") (net 3))
   (segment (start 164.75 102) (end 163.25 100.7) (width 0.2) (layer "B.Cu") (net 3))
   (segment (start 140.2 103.95) (end 140.2 102.8) (width 0.5) (layer "B.Cu") (net 3))
@@
   (segment (start 157.3 99.1) (end 158.9 100.7) (width 0.5) (layer "B.Cu") (net 3))
   (segment (start 158.9 100.7) (end 163.25 100.7) (width 0.5) (layer "B.Cu") (net 3))
+  (segment (start 141.3 101.7) (end 143.8 101.7) (width 0.5) (layer "B.Cu") (net 3))
+  (segment (start 141.55 98.5375) (end 143.1375 98.5375) (width 0.5) (layer "B.Cu") (net 3))
   (segment (start 152.765 97.635) (end 151.9 98.5) (width 0.5) (layer "B.Cu") (net 3))
+  (segment (start 143.1375 98.5375) (end 143.8 99.2) (width 0.5) (layer "B.Cu") (net 3))
   (segment (start 153.725 97.635) (end 152.765 97.635) (width 0.5) (layer "B.Cu") (net 3))
+  (segment (start 143.8 101.7) (end 151 101.7) (width 0.5) (layer "B.Cu") (net 3))
   (segment (start 153.725 97.635) (end 155.835 97.635) (width 0.5) (layer "B.Cu") (net 3))
   (segment (start 174.5 98.75) (end 170.5 98.75) (width 0.2) (layer "B.Cu") (net 4))
@@
   (segment (start 138.2 102.4) (end 139.8 100.8) (width 0.5) (layer "B.Cu") (net 4))
   (segment (start 166.05 98.8) (end 163.25 98.8) (width 0.2) (layer "B.Cu") (net 4))
+  (segment (start 139.65 98.5375) (end 139.65 100.65) (width 0.5) (layer "B.Cu") (net 4))
   (segment (start 167.5 99.44) (end 166.05 98.8) (width 0.2) (layer "B.Cu") (net 4))
   (segment (start 169.81 99.44) (end 167.5 99.44) (width 0.2) (layer "B.Cu") (net 4))
@@
   (segment (start 151.2 97.915001) (end 152.750001 96.365) (width 0.5) (layer "B.Cu") (net 4))
   (segment (start 138.2 103.95) (end 138.2 102.4) (width 0.5) (layer "B.Cu") (net 4))
+  (segment (start 139.65 100.65) (end 139.8 100.8) (width 0.5) (layer "B.Cu") (net 4))
   (segment (start 151.2 100) (end 151.2 97.915001) (width 0.5) (layer "B.Cu") (net 4))
   (segment (start 166.54 98.29) (end 163.13 94.88) (width 0.5) (layer "F.Cu") (net 6))

Commit message: schematic and pcb bug fix for Vcc and Vio swap on CAN xcvr
Parts:
- moved C3 13.8 mm to (144.4, 95.8), turned to 180 degrees
- moved C2 13.2 mm to (158.4, 94.8), turned to 0 degrees
Connections:
- U2 pad 3: +3.3V -> +5V
- U2 pad 5: +5V -> +3.3V
Routing:
- net +5V: track 18.0 -> 27.7 mm
- net +3.3V: track 17.2 -> 10.6 mm
- net GND: vias 22 -> 25
Changed lines of the file:
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@@
   )
   (footprint "Capacitor_SMD:C_0805_2012Metric_Pad1.18x1.45mm_HandSolder" (layer "B.Cu")
-    (at 158.2 95.4)
+    (at 144.4 95.8 180)
     (descr "Capacitor SMD 0805 (2012 Metric), square (rectangular) end terminal, IPC_7351 nominal with elongated pad for handsoldering. (Body size source: IPC-SM-782 page 76, https://www.pcb-3d.com/wordpress/wp-content/uploads/ipc-sm-782a_amendment_1_and_2.pdf, https://docs.google.com/spreadsheets/d/1BsfQQcO9C6DZCsRaXUlFlo91Tg2WpOkGARC1WS5S8t0/edit?usp=sharing), generated with kicad-footprint-generator")
     (tags "capacitor handsolder")
@@
     (fp_line (start 1 0.625) (end 1 -0.625)
       (stroke (width 0.1) (type solid)) (layer "B.Fab"))
-    (pad "1" smd roundrect (at -1.0375 0) (size 1.175 1.45) (layers "B.Cu" "B.Paste" "B.Mask") (roundrect_rratio 0.212766)
+    (pad "1" smd roundrect (at -1.0375 0 180) (size 1.175 1.45) (layers "B.Cu" "B.Paste" "B.Mask") (roundrect_rratio 0.212766)
       (net 6 "+5V") (pintype "passive"))
-    (pad "2" smd roundrect (at 1.0375 0) (size 1.175 1.45) (layers "B.Cu" "B.Paste" "B.Mask") (roundrect_rratio 0.212766)
+    (pad "2" smd roundrect (at 1.0375 0 180) (size 1.175 1.45) (layers "B.Cu" "B.Paste" "B.Mask") (roundrect_rratio 0.212766)
       (net 2 "GND") (pintype "passive"))
     (model "${KICAD6_3DMODEL_DIR}/Capacitor_SMD.3dshapes/C_0805_2012Metric.wrl"
@@
       (net 2 "GND") (pinfunction "GND") (pintype "power_in"))
     (pad "3" smd roundrect (at -2.475 -0.635) (size 1.95 0.6) (layers "B.Cu" "B.Paste" "B.Mask") (roundrect_rratio 0.25)
-      (net 19 "+3.3V") (pinfunction "VCC") (pintype "power_in"))
+      (net 6 "+5V") (pinfunction "VCC") (pintype "power_in"))
     (pad "4" smd roundrect (at -2.475 -1.905) (size 1.95 0.6) (layers "B.Cu" "B.Paste" "B.Mask") (roundrect_rratio 0.25)
       (net 21 "/CAN_RXD") (pinfunction "RXD") (pintype "output"))
     (pad "5" smd roundrect (at 2.475 -1.905) (size 1.95 0.6) (layers "B.Cu" "B.Paste" "B.Mask") (roundrect_rratio 0.25)
-      (net 6 "+5V") (pinfunction "VIO") (pintype "power_in"))
+      (net 19 "+3.3V") (pinfunction "VIO") (pintype "power_in"))
     (pad "6" smd roundrect (at 2.475 -0.635) (size 1.95 0.6) (layers "B.Cu" "B.Paste" "B.Mask") (roundrect_rratio 0.25)
       (net 4 "/CANL") (pinfunction "CANL") (pintype "bidirectional"))
@@
   )
   (footprint "Capacitor_SMD:C_0805_2012Metric_Pad1.18x1.45mm_HandSolder" (layer "B.Cu")
-    (at 145.2 95 180)
+    (at 158.4 94.8)
     (descr "Capacitor SMD 0805 (2012 Metric), square (rectangular) end terminal, IPC_7351 nominal with elongated pad for handsoldering. (Body size source: IPC-SM-782 page 76, https://www.pcb-3d.com/wordpress/wp-content/uploads/ipc-sm-782a_amendment_1_and_2.pdf, https://docs.google.com/spreadsheets/d/1BsfQQcO9C6DZCsRaXUlFlo91Tg2WpOkGARC1WS5S8t0/edit?usp=sharing), generated with kicad-footprint-generator")
     (tags "capacitor handsolder")
@@
     (fp_line (start 1 0.625) (end 1 -0.625)
       (stroke (width 0.1) (type solid)) (layer "B.Fab"))
-    (pad "1" smd roundrect (at -1.0375 0 180) (size 1.175 1.45) (layers "B.Cu" "B.Paste" "B.Mask") (roundrect_rratio 0.212766)
+    (pad "1" smd roundrect (at -1.0375 0) (size 1.175 1.45) (layers "B.Cu" "B.Paste" "B.Mask") (roundrect_rratio 0.212766)
       (net 19 "+3.3V") (pintype "passive"))
-    (pad "2" smd roundrect (at 1.0375 0 180) (size 1.175 1.45) (layers "B.Cu" "B.Paste" "B.Mask") (roundrect_rratio 0.212766)
+    (pad "2" smd roundrect (at 1.0375 0) (size 1.175 1.45) (layers "B.Cu" "B.Paste" "B.Mask") (roundrect_rratio 0.212766)
       (net 2 "GND") (pintype "passive"))
     (model "${KICAD6_3DMODEL_DIR}/Capacitor_SMD.3dshapes/C_0805_2012Metric.wrl"
@@
   (segment (start 165.25 92.5) (end 165.25 90.2875) (width 0.5) (layer "F.Cu") (net 1))
   (segment (start 165.25 90.2875) (end 164.7125 89.75) (width 0.5) (layer "F.Cu") (net 1))
+  (via (at 146.2 94) (size 0.8) (drill 0.4) (layers "F.Cu" "B.Cu") (free) (net 2))
   (via (at 137 109.6) (size 0.8) (drill 0.4) (layers "F.Cu" "B.Cu") (free) (net 2))
   (via (at 155.4 103.8) (size 0.8) (drill 0.4) (layers "F.Cu" "B.Cu") (free) (net 2))
@@
   (via (at 149.4 104.4) (size 0.8) (drill 0.4) (layers "F.Cu" "B.Cu") (free) (net 2))
   (via (at 131.2 104.2) (size 0.8) (drill 0.4) (layers "F.Cu" "B.Cu") (free) (net 2))
+  (via (at 165.8 95.2) (size 0.8) (drill 0.4) (layers "F.Cu" "B.Cu") (free) (net 2))
+  (via (at 162.4 96.6) (size 0.8) (drill 0.4) (layers "F.Cu" "B.Cu") (free) (net 2))
   (via (at 162.5 92) (size 0.8) (drill 0.4) (layers "F.Cu" "B.Cu") (free) (net 2))
   (via (at 135.25 94) (size 0.8) (drill 0.4) (layers "F.Cu" "B.Cu") (free) (net 2))
@@
   (segment (start 163.13 94.88) (end 158.89 94.88) (width 0.5) (layer "F.Cu") (net 6))
   (segment (start 168.5 98.29) (end 166.54 98.29) (width 0.5) (layer "F.Cu") (net 6))
-  (segment (start 155.72 94.88) (end 155.6 95) (width 0.5) (layer "F.Cu") (net 6))
-  (segment (start 158.89 94.88) (end 155.72 94.88) (width 0.5) (layer "F.Cu") (net 6))
-  (via (at 155.6 95) (size 0.8) (drill 0.4) (layers "F.Cu" "B.Cu") (net 6))
-  (segment (start 155.505 95.095) (end 155.6 95) (width 0.5) (layer "B.Cu") (net 6))
-  (segment (start 156 95.4) (end 155.6 95) (width 0.5) (layer "B.Cu") (net 6))
-  (segment (start 153.725 95.095) (end 155.505 95.095) (width 0.5) (layer "B.Cu") (net 6))
-  (segment (start 157.1625 95.4) (end 156 95.4) (width 0.5) (layer "B.Cu") (net 6))
+  (segment (start 158.89 94.88) (end 158.21 94.2) (width 0.5) (layer "F.Cu") (net 6))
+  (segment (start 158.21 94.2) (end 149.165 94.2) (width 0.5) (layer "F.Cu") (net 6))
+  (segment (start 149.165 94.2) (end 147 96.365) (width 0.5) (layer "F.Cu") (net 6))
+  (via (at 147 96.365) (size 0.8) (drill 0.4) (layers "F.Cu" "B.Cu") (net 6))
+  (segment (start 146.0025 96.365) (end 147 96.365) (width 0.5) (layer "B.Cu") (net 6))
+  (segment (start 145.4375 95.8) (end 146.0025 96.365) (width 0.5) (layer "B.Cu") (net 6))
+  (segment (start 147 96.365) (end 148.775 96.365) (width 0.5) (layer "B.Cu") (net 6))
   (segment (start 133.6 100.2) (end 133.6 97.2275) (width 0.5) (layer "B.Cu") (net 7))
   (segment (start 133.6 97.2275) (end 133.5925 97.22) (width 0.5) (layer "B.Cu") (net 7))
@@
   (segment (start 164.34 105.91) (end 160.13 110.12) (width 0.5) (layer "F.Cu") (net 15))
   (segment (start 160.13 110.12) (end 158.89 110.12) (width 0.5) (layer "F.Cu") (net 15))
-  (segment (start 147.11875 95.88125) (end 148.6375 97.4) (width 0.5) (layer "F.Cu") (net 19))
-  (segment (start 155.33 97.4) (end 157.89 99.96) (width 0.5) (layer "F.Cu") (net 19))
+  (segment (start 155.4 95.5155) (end 155.4 97.47) (width 0.5) (layer "F.Cu") (net 19))
+  (segment (start 155.4 97.47) (end 157.89 99.96) (width 0.5) (layer "F.Cu") (net 19))
   (segment (start 157.89 99.96) (end 158.89 99.96) (width 0.5) (layer "F.Cu") (net 19))
-  (segment (start 148.6375 97.4) (end 155.33 97.4) (width 0.5) (layer "F.Cu") (net 19))
-  (via (at 147.11875 95.88125) (size 0.8) (drill 0.4) (layers "F.Cu" "B.Cu") (net 19))
-  (segment (start 147.11875 95.88125) (end 147.6025 96.365) (width 0.5) (layer "B.Cu") (net 19))
-  (segment (start 148.775 96.365) (end 147.6025 96.365) (width 0.5) (layer "B.Cu") (net 19))
-  (segment (start 147.6025 96.365) (end 146.2375 95) (width 0.5) (layer "B.Cu") (net 19))
+  (via (at 155.4 95.5155) (size 0.8) (drill 0.4) (layers "F.Cu" "B.Cu") (net 19))
+  (segment (start 155.4 95.5155) (end 154.9795 95.095) (width 0.5) (layer "B.Cu") (net 19))
+  (segment (start 156.1155 94.8) (end 155.4 95.5155) (width 0.5) (layer "B.Cu") (net 19))
+  (segment (start 154.9795 95.095) (end 153.725 95.095) (width 0.5) (layer "B.Cu") (net 19))
+  (segment (start 157.3625 94.8) (end 156.1155 94.8) (width 0.5) (layer "B.Cu") (net 19))
   (segment (start 147.55 99.95) (end 142.46 105.04) (width 0.5) (layer "F.Cu") (net 20))
   (segment (start 142.46 105.04) (end 141.11 105.04) (width 0.5) (layer "F.Cu") (net 20))
